File: PCB/electronix.kicad_sch (KiCad schematic)
At the start: 132 parts, among them IC1 ICM-20602, IC2 AP9101CK6-ANTRG1, IC3 DRV8210DRLR, IC4 DRV8210DRLR, IC5 LM66200DRLR, J1 USB-C 6pin, J2 PRG, M1 N20, M2 N20, Q1 UMH3N FHA, Q2 dual NMOS, Q3 dual NMOS, Q4 Phototransistor, Q5 Phototransistor, Q6 dual NMOS, Q7 Phototransistor, Q8 Phototransistor, SW1 side slide, SW2 RESET, SW3 START, U1 MCP73213-A6SI/MF, U2 ESP32-WROOM-32, U3 LMR51420YDDRCR

Commit message: Update ibom.html, electronix.kicad_pcb, and electronix.kicad_sch
Parts:
- renumbered IC1 to ICe
Changed lines of the file:
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@@
       (effects (font (size 1.27 1.27)) (justify bottom) hide)
     )
-    (property "Datasheet" "" (at 113.03 196.85 0)
+    (property "Datasheet" "https://ww1.microchip.com/downloads/en/DeviceDoc/20002190C.pdf" (at 113.03 196.85 0)
       (effects (font (size 1.27 1.27)) hide)
     )
@@
   (symbol (lib_id "ICM-20602:ICM-20602") (at 77.47 57.15 0) (unit 1)
     (in_bom yes) (on_board yes) (dnp no) (fields_autoplaced)
-    (property "Reference" "IC1" (at 66.04 39.37 0)
+    (property "Reference" "ICe" (at 66.04 39.37 0)
       (effects (font (size 1.27 1.27)) (justify left))
     )
@@
       (effects (font (size 1.27 1.27)) (justify left) hide)
     )
-    (property "Datasheet" "https://3cfeqx1hf82y3xcoull08ihx-wpengine.netdna-ssl.com/wp-content/uploads/2021/03/DS-000135-ICG-20660-TYP-v1.2.pdf" (at 73.66 36.83 0)
+    (property "Datasheet" "https://invensense.tdk.com/wp-content/uploads/2020/11/DS-000176-ICM-20602-v1.1.pdf" (at 73.66 36.83 0)
       (effects (font (size 1.27 1.27)) (justify left) hide)
     )
@@
       (project "electronix"
         (path "/eef2ed29-f372-440b-8687-49cc4274d156"
-          (reference "IC1") (unit 1)
-        )
-      )
+          (reference "ICe") (unit 1)
+        )
+      )
